File: kicad/CoCoTANG.kicad_sch (KiCad schematic)
At the start: 105 parts, among them J1 CPU, J10 PIA0, J11 PIA1, J12 PIA1_SOCKET, J13 ADDRMUX_SOCKET, J14 PIA0, J15 PIA1, J16 VDG_IN, J17 AV_IN, J18 CMP_IN, J19 VDG_OUT, J2 ADDRMUX, J20 AV_OUT, J21 CMP_OUT, J3 CPU_SOCKET, J4 PIA0, J5 PIA1, J6 ADDRMUX, J7 AV_HEADER, J8 ADDRMUX, J9 PIA0_SOCKET, Q1 2N3904, Q2 2N3904, Q3 2N3904, Q4 MMBT3904, Q5 MMBT3904, Q6 MMBT3904, Q7 MMBT3904, Q8 MMBT3904, Q9 MMBT3904, U10 SN74LVC245AN, U11 SN74LVC245AN, U12 SN74LVC245AN, U3 74HC139, U5 Tang_Nano_20k, U7 74HC30, U8 SN74LVC245AN, U9 SN74LVC245AN

Commit message: changes
Parts:
- removed J19: VDG_OUT, Connector_PinHeader_2.54mm:PinHeader_1x05_P2.54mm_Vertical, symbol Connector_Generic:Conn_01x05
- removed J2, J8: ADDRMUX, Connector_PinHeader_2.54mm:PinHeader_1x05_P2.54mm_Vertical, symbol Connector_Generic:Conn_01x05
- removed Q1, Q2, Q3: 2N3904, Package_TO_SOT_SMD:SOT-23, symbol Transistor_BJT:2N3904
- added C32: 104, Capacitor_SMD:C_0805_2012Metric_Pad1.18x1.45mm_HandSolder, symbol Device:C
- added D1, D3: BAT54H,111, Diode_SMD:D_SOD-123F, symbol Device:D_Schottky
- added J19: ADDRMUX, Connector_PinSocket_2.54mm:PinSocket_1x07_P2.54mm_Vertical, symbol Connector_Generic:Conn_01x07
- added J22: 74HC11, Package_SO:TSSOP-14_4.4x5mm_P0.65mm, symbol Connector_Generic:Conn_02x07_Counter_Clockwise
- added J23: TRG, Connector_PinHeader_2.54mm:PinHeader_1x02_P2.54mm_Vertical, symbol Connector_Generic:Conn_01x02
- added J24: VDG_SOCKET, Package_DIP:DIP-40_W15.24mm_Socket, symbol Connector_Generic:Conn_02x20_Counter_Clockwise
- added J25: AUDIO_OUT, Connector_PinHeader_2.54mm:PinHeader_1x02_P2.54mm_Vertical, symbol Connector_Generic:Conn_01x02
- added J8: ADDRMUX, Package_DFN_QFN:QFN-20-1EP_5x5mm_P0.65mm_EP3.35x3.35mm, symbol Connector_Generic:Conn_01x07
- added Q10, Q11, Q12: 2N3904, Package_TO_SOT_SMD:SOT-23, symbol Transistor_BJT:Q_NPN_CBE
- added RV1: VREF, FPGA_Common:PVG3G_BRN, symbol Device:R_Potentiometer_US
- U9: value SN74LVC245AN -> SN74HC245PWR
Connections:
- net +5V: now also C32.1, J22.14 (Pin_14), J24.17 (Pin_17), RV1.1
- net AUDIO_RCA: now also J25.1 (Pin_1)
- net CVBS_33: now also J7.2 (Pin_2), U5.33 (54_IOR38A)
- net D0: now also J1.31 (Pin_31), J3.31 (Pin_31); no longer J1.24 (Pin_24), J3.24 (Pin_24)
- net D1: now also J1.30 (Pin_30), J3.30 (Pin_30); no longer J1.25 (Pin_25), J3.25 (Pin_25)
- net D2: now also J1.29 (Pin_29), J3.29 (Pin_29); no longer J1.26 (Pin_26), J3.26 (Pin_26)
- net D3: now also J1.28 (Pin_28), J3.28 (Pin_28); no longer J1.27 (Pin_27), J3.27 (Pin_27)
- net D4: now also J1.27 (Pin_27), J3.27 (Pin_27); no longer J1.28 (Pin_28), J3.28 (Pin_28)
- net D5: now also J1.26 (Pin_26), J3.26 (Pin_26); no longer J1.29 (Pin_29), J3.29 (Pin_29)
- net D6: now also J1.25 (Pin_25), J3.25 (Pin_25); no longer J1.30 (Pin_30), J3.30 (Pin_30)
- net D7: now also J1.24 (Pin_24), J3.24 (Pin_24); no longer J1.31 (Pin_31), J3.31 (Pin_31)
- net E_33: now also U5.32 (51_IOR45A); no longer U5.3 (75_IOT34A)
- net GND: now also C32.2, J22.7 (Pin_7), J24.1 (Pin_1), J25.2 (Pin_2), Q10.3 (E), Q11.3 (E), Q12.3 (E), RV1.3
- net PB_33: no longer J7.2 (Pin_2), U5.33 (54_IOR38A)
- net PIA0: now also J22.11 (Pin_11), J22.4 (Pin_4)
- net PIA1: now also J22.10 (Pin_10), J22.5 (Pin_5)
- net PR_33: no longer U5.32 (51_IOR45A)
- net ROW0: now also D1.2 (A)
- net ROW1: now also D3.2 (A)
- net R/~{W}: now also J19.6 (Pin_6), J22.9 (Pin_9), J8.6 (Pin_6); no longer U12.1 (A->B)
- net S0: now also J19.1 (Pin_1), J8.1 (Pin_1)
- net S1: now also J19.2 (Pin_2), J8.2 (Pin_2)
- net S2: now also J19.3 (Pin_3), J8.3 (Pin_3)
- net Y_VDG: now also J24.28 (Pin_28)
- net ~{EXTROM}: now also J22.13 (Pin_13)
- net ~{FIRQ}: now also Q12.1 (C)
- net ~{HALT}: now also Q11.1 (C)
- net ~{IRQ}: now also Q10.1 (C)
- net ~{MRD}: now also J22.1 (Pin_1); no longer U12.19 (CE)
- net ~{ROM}: now also J22.2 (Pin_2)
- net ~{SLENB}: now also J19.5 (Pin_5), J8.5 (Pin_5)
- net at R5.1: now also Q11.2 (B)
- net at R7.1: now also Q12.2 (B)
- net at R3.1: now also Q10.2 (B)
- net CHA_VDG renamed CLRA
- net CLRA: now also J24.11 (Pin_11)
- net CHB_VDG renamed CLRB
- net CLRB: now also J24.10 (Pin_10)
- net HALT_33 renamed RESET_33
- new net: D3.1 (K), J23.2 (Pin_2)
- new net: D1.1 (K), J23.1 (Pin_1)
- new net CHB: J24.9 (Pin_9), RV1.2
- new net DATADIR: J19.7 (Pin_7), J22.8 (Pin_8), J8.7 (Pin_7), U12.1 (A->B)
- new net ~{DATAEN}: J19.4 (Pin_4), J22.6 (Pin_6), J8.4 (Pin_4), U12.19 (CE)
- new net ~{MENEN}: J22.12 (Pin_12), J22.3 (Pin_3)
- no-connect marks 17 -> 52
Other:
- moved on the sheet: C1, C17, C18, C19, C20, C21, J12, J13, J14, J15, J16, J4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

Commit message: new board
Parts:
- removed C10, C12: 22uF, Capacitor_SMD:C_0805_2012Metric_Pad1.18x1.45mm_HandSolder, symbol Device:C
- removed C17, C18, C19: 68pF, Capacitor_SMD:C_0805_2012Metric_Pad1.18x1.45mm_HandSolder, symbol Device:C
- removed C20: 4.7uF, Capacitor_SMD:C_0805_2012Metric_Pad1.18x1.45mm_HandSolder, symbol Device:C
- removed C21: 6.8nF, Capacitor_SMD:C_0805_2012Metric_Pad1.18x1.45mm_HandSolder, symbol Device:C
- removed J10, J14: PIA0, Connector_PinHeader_2.54mm:PinHeader_1x03_P2.54mm_Vertical, symbol Connector_Generic:Conn_01x03
- removed J11, J15: PIA1, Connector_PinHeader_2.54mm:PinHeader_1x02_P2.54mm_Vertical, symbol Connector_Generic:Conn_01x02
- removed J13: ADDRMUX_SOCKET, Package_DIP:DIP-16_W7.62mm_Socket, symbol Connector_Generic:Conn_02x08_Counter_Clockwise
- removed J16: VDG_IN, Connector_PinHeader_2.54mm:PinHeader_1x06_P2.54mm_Vertical, symbol Connector_Generic:Conn_01x06
- removed J19: ADDRMUX, Connector_PinSocket_2.54mm:PinSocket_1x07_P2.54mm_Vertical, symbol Connector_Generic:Conn_01x07
- removed J24: VDG_SOCKET, Package_DIP:DIP-40_W15.24mm_Socket, symbol Connector_Generic:Conn_02x20_Counter_Clockwise
- removed J25: AUDIO_OUT, Connector_PinHeader_2.54mm:PinHeader_1x02_P2.54mm_Vertical, symbol Connector_Generic:Conn_01x02
- removed J6: ADDRMUX, Package_DIP:DIP-16_W7.62mm_Socket, symbol Connector_Generic:Conn_02x08_Counter_Clockwise
- removed J8: ADDRMUX, Package_DFN_QFN:QFN-20-1EP_5x5mm_P0.65mm_EP3.35x3.35mm, symbol Connector_Generic:Conn_01x07
- removed Q10, Q11, Q12: 2N3904, Package_TO_SOT_SMD:SOT-23, symbol Transistor_BJT:Q_NPN_CBE
- removed Q4, Q5, Q6, Q7, Q8, Q9: MMBT3904, Package_TO_SOT_SMD:SOT-23, symbol Transistor_BJT:MMBT3904
- removed R19, R20, R21: 100, Resistor_SMD:R_0805_2012Metric_Pad1.20x1.40mm_HandSolder, symbol Device:R
- removed RV1: VREF, FPGA_Common:PVG3G_BRN, symbol Device:R_Potentiometer_US
- added C33: 104, Capacitor_SMD:C_0805_2012Metric_Pad1.18x1.45mm_HandSolder, symbol Device:C
- added J2: CPU_SOCKET_ZIF, FPGA_Common:CONN_CF4240FH0R0-05-NH_CVI, symbol FPGA_Common:CF4240FH0R0-05-NH
- added J22: PIA0_SOCKET_ZIF, FPGA_Common:CONN_CF4240FH0R0-05-NH_CVI, symbol FPGA_Common:CF4240FH0R0-05-NH
- added J24: PIA0_ZIF, FPGA_Common:CONN_CF4240FH0R0-05-NH_CVI, symbol FPGA_Common:CF4240FH0R0-05-NH
- added J26: PIA1_SOCKET_ZIF, FPGA_Common:CONN_CF4240FH0R0-05-NH_CVI, symbol FPGA_Common:CF4240FH0R0-05-NH
- added J27: ADDRMUX_SOCKET_ZIF, FPGA_Common:CONN_CF4216FH0R0-05-NH_CVI, symbol FPGA_Common:5034801600
- added J28: ADDRMUX_SOCKET, Package_DIP:DIP-16_W7.62mm_Socket, symbol Connector_Generic:Conn_02x08_Counter_Clockwise
- added J29: PIA1_ZIF, FPGA_Common:CONN_CF4240FH0R0-05-NH_CVI, symbol FPGA_Common:CF4240FH0R0-05-NH
- added J30: ADDRMUX_ZIF, FPGA_Common:CONN_CF4216FH0R0-05-NH_CVI, symbol FPGA_Common:5034801600
- added J6: CLK, Connector_PinSocket_2.54mm:PinSocket_1x01_P2.54mm_Vertical, symbol Connector_Generic:Conn_01x01
- added J8: CPU_ZIF, FPGA_Common:CONN_CF4240FH0R0-05-NH_CVI, symbol FPGA_Common:CF4240FH0R0-05-NH
- added Q1, Q2, Q3, Q4, Q5, Q6, Q7, Q8, Q9: MMBT3904-TP, FPGA_Common:SOT-23_MCC, symbol FPGA_Common:MMBT3904-TP
- added R1, R37, R38, R39: 1K, Resistor_SMD:R_0805_2012Metric_Pad1.20x1.40mm_HandSolder, symbol Device:R
- added U1: SN74HC138PWR, Package_SO:TSSOP-16_4.4x5mm_P0.65mm, symbol FPGA_Common:SN74HC138PWR
- C14: value 680pF -> 470pF
- R17: value 100K -> 1K
- renumbered J22 to U22
Connections:
- net +3.3V: now also Q1.3, Q2.3, Q3.3, Q4.3, Q5.3, Q6.3; no longer C2.1, U9.20 (VCC)
- net +5V: now also C2.1, U9.20 (VCC), C33.1, J2.7, J22.20, J24.20, J26.20, J27.13, J27.14, J27.15, J27.16, J28.13 (Pin_13), J28.14 (Pin_14), J28.15 (Pin_15), J28.16 (Pin_16), J29.20, J30.13, J30.14, J30.15, J30.16, J8.7, U1.16 (VCC)
- net A0: now also J2.8, J8.8
- net A1: now also J2.9, J8.9
- net A10: now also J2.18, J8.18
- net A11: now also J2.19, J8.19
- net A12: now also J2.20, J8.20
- net A13: now also J2.21, J8.21
- net A14: now also J2.22, J8.22
- net A15: now also J2.23, J8.23
- net A2: now also J2.10, J8.10
- net A3: now also J2.11, J8.11
- net A4: now also J2.12, J8.12
- net A5: now also J2.13, J8.13
- net A6: now also J2.14, J8.14
- net A7: now also J2.15, J8.15
- net A8: now also J2.16, J8.16
- net A9: now also J2.17, J8.17
- net AP10: now also J22.10, J24.10
- net AP11: now also J22.11, J24.11
- net AP12: now also J22.12, J24.12
- net AP13: now also J22.13, J24.13
- net AP14: now also J22.14, J24.14
- net AP15: now also J22.15, J24.15
- net AP16: now also J22.16, J24.16
- net AP17: now also J22.17, J24.17
- net AP18: now also J22.19, J24.19
- net AP21: now also J22.21, J24.21
- net AP22: now also J22.22, J24.22
- net AP23: now also J22.23, J24.23
- net AP24: now also J22.24, J24.24
- net AP25: now also J22.25, J24.25
- net AP26: now also J22.26, J24.26
- net AP27: now also J22.27, J24.27
- net AP28: now also J22.28, J24.28
- net AP29: now also J22.29, J24.29
- net AP30: now also J22.30, J24.30
- net AP31: now also J22.31, J24.31
- net AP32: now also J22.32, J24.32
- net AP33: now also J22.33, J24.33
- net AP34: now also J22.34, J24.34
- net AP35: now also J22.35, J24.35
- net AP36: now also J22.36, J24.36
- net AP37: now also J22.37, J24.37
- net AP38: now also J22.38, J24.38
- net AP39: now also J22.39, J24.39
- net AP9: now also J22.9, J24.9
- net AUDIO_33: now also U9.9 (A7); no longer R16.1
- net AUDIO_RCA: no longer R17.2
- net BP11: now also J26.11, J29.11
- net BP12: now also J26.12, J29.12
- net BP13: now also J26.13, J29.13
- net BP14: now also J26.14, J29.14
- net BP15: now also J26.15, J29.15
- net BP16: now also J26.16, J29.16
- net BP17: now also J26.17, J29.17
- net BP19: now also J26.19, J29.19
- net BP2: now also J26.2, J29.2
- net BP21: now also J26.21, J29.21
- net BP22: now also J26.22, J29.22
- net BP23: now also J26.23, J29.23
- net BP24: now also J26.24, J29.24
- net BP25: now also J26.25, J29.25
- net BP26: now also J26.26, J29.26
- net BP27: now also J26.27, J29.27
- net BP28: now also J26.28, J29.28
- net BP29: now also J26.29, J29.29
- net BP3: now also J26.3, J29.3
- net BP30: now also J26.30, J29.30
- net BP31: now also J26.31, J29.31
- net BP32: now also J26.32, J29.32
- net BP33: now also J26.33, J29.33
- net BP34: now also J26.34, J29.34
- net BP35: now also J26.35, J29.35
- net BP36: now also J26.36, J29.36
- net BP37: now also J26.37, J29.37
- net BP38: now also J26.38, J29.38
- net BP39: now also J26.39, J29.39
- net BP4: now also J26.4, J29.4
- net BP40: now also J26.40, J29.40
- net BP5: now also J26.5, J29.5
- net BP6: now also J26.6, J29.6
- net BP7: now also J26.7, J29.7
- net BP8: now also J26.8, J29.8
- net BP9: now also J26.9, J29.9
- net CP33: now also J2.33, J8.33
- net CP36: now also J2.36, J8.36
- net CP38: now also J2.38, J8.38
- net CP39: now also J2.39, J8.39
- net CP5: now also J2.5, J8.5
- net CP6: now also J2.6, J8.6
- net CVBS_33: now also J7.3 (Pin_3), U5.18 (18_IOL49B_LED3); no longer J7.2 (Pin_2), U5.33 (54_IOR38A)
- net D0: now also J2.31, J8.31
- net D1: now also J2.30, J8.30
- net D2: now also J2.29, J8.29
- net D3: now also J2.28, J8.28
- net D4: now also J2.27, J8.27
- net D5: now also J2.26, J8.26
- net D6: now also J2.25, J8.25
- net D7: now also J2.24, J8.24
- net DP4: now also J27.4, J28.4 (Pin_4), J30.4, U1.4 (*G2A)
- net DP5: now also J27.5, J28.5 (Pin_5), J30.5, U1.5 (*G2B)
- net E: now also J2.34, J8.34
- net FIRQ_33: now also U5.3 (75_IOT34A); no longer U5.18 (18_IOL49B_LED3)
- net GND: now also R16.2, R17.2, C33.2, J2.1, J22.1, J24.1, J26.1, J27.8, J28.8 (Pin_8), J29.1, J30.8, J8.1, Q7.2, Q8.2, Q9.2, R1.2, R37.2, R38.2, R39.2, U1.8 (GND); no longer R17.1
- net PB_RCA: now also R11.2
- net PIA0: now also J27.11, J28.11 (Pin_11), J30.11, U1.11 (Y4)
- net PIA1: now also J27.10, J28.10 (Pin_10), J30.10, U1.10 (Y5)
- net PR_33: no longer J7.3 (Pin_3)
- net PR_RCA: now also R12.2
- net Q: now also J2.35, J8.35
- net ROW0: now also J22.2, J24.2
- net ROW1: now also J22.3, J24.3
- net ROW2: now also J22.4, J24.4
- net ROW3: now also J22.5, J24.5
- net ROW4: now also J22.6, J24.6
- net ROW5: now also J22.7, J24.7
- net ROW6: now also J22.8, J24.8
- net R/~{W}: now also J2.32, J8.32
- net S0: now also J27.1, J28.1 (Pin_1), J30.1, U1.1 (A)
- net S1: now also J27.2, J28.2 (Pin_2), J30.2, U1.2 (B)
- net S2: now also J27.3, J28.3 (Pin_3), J30.3, U1.3 (C)
- net SERNT: now also J26.10, J29.10
- net ~{CART}: now also J26.18, J29.18
- net ~{CTS}: now also J27.12, J28.12 (Pin_12), J30.12, U1.12 (Y3)
- net ~{EXTROM}: now also U1.13 (Y2)
- net ~{FIRQ}: now also J2.4, J8.4, Q8.3
- net ~{FS}: now also J22.18, J24.18
- net ~{HALT}: now also J2.40, J8.40, Q9.3
- net ~{HS}: now also J22.40, J24.40
- net ~{IRQ}: now also J2.3, J8.3, Q7.3
- net ~{MRD}: now also U1.15 (Y0)
- net ~{NMI}: now also J2.2, J8.2
- net ~{RESET}: now also J2.37, J8.37
- net ~{ROM}: now also U1.14 (Y1)
- net ~{SCS}: now also J27.9, J28.9 (Pin_9), J30.9, U1.9 (Y6)
- net ~{SLENB}: now also J27.6, J28.6 (Pin_6), J30.6, U1.6 (G1)
- net at R29.2, R30.1: now also Q6.1
- net at R15.1: now also Q6.2, R39.1
- net at R35.2, R36.1: now also Q5.1
- net at R31.2, R32.1: now also Q2.1
- net at R5.1: now also Q9.1
- net CLK: now reaches U9.11 (B7)
- net CLK: now also J6.1 (Pin_1)
- net at R11.1: now also Q4.2, R1.1
- net at R25.2, R26.1: now also Q1.1
- net at R33.2, R34.1: now also Q4.1
- net at R13.2: now also Q1.2, R38.1
- net at R7.1: now also Q8.1
- net at R12.1: now also R16.1, Q5.2
- net at R10.1: now also R17.1, Q2.2
- net at R3.1: now also Q7.1
- net at R27.2, R28.1: now also Q3.1
- net at R14.2: now also Q3.2, R37.1
- new net CHR_33: J7.2 (Pin_2), U5.33 (54_IOR38A)
- no-connect marks 52 -> 21
Other:
- note added: "ADDRMUX DISPLACER"
- note added: "CPU DISPLACER"
- note removed: "ADDR MUX DISPLACER"
- note removed: "VDG HAT"
- moved on the sheet: C1, C11, C13, C14, C15, C16, C2, C22, C23, C24, C25, C26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

Commit message: fixes
Parts:
- removed J27: ADDRMUX_SOCKET_ZIF, FPGA_Common:CONN_CF4216FH0R0-05-NH_CVI, symbol FPGA_Common:5034801600
- removed J30: ADDRMUX_ZIF, FPGA_Common:CONN_CF4216FH0R0-05-NH_CVI, symbol FPGA_Common:5034801600
- added C34: 104, Capacitor_SMD:C_0805_2012Metric_Pad1.18x1.45mm_HandSolder, symbol Device:C
- added H1, H2, H3, H4: MountingHole, MountingHole:MountingHole_3mm, symbol Mechanical:MountingHole
- added J10: 74LS138_ZIF, FPGA_Common:CONN_CF4216FH0R0-05-NH_CVI, symbol FPGA_Common:CF4216FH0R0-05-NH
- added J11: 74LS138_ZIF_SOCKET, FPGA_Common:CONN_CF4216FH0R0-05-NH_CVI, symbol FPGA_Common:CF4216FH0R0-05-NH
- added J13: CoCo_Cart, FPGA_Common:COCO_CART, symbol FPGA_Common:CoCo_Cart
- added JP1: Jumper_2_Open, Jumper:SolderJumper-2_P1.3mm_Open_Pad1.0x1.5mm, symbol Jumper:Jumper_2_Open
- added U2: AT28C64B-15PU, FPGA_Common:28P6_ATM, symbol FPGA_Common:AT28C64B-15PU
Connections:
- net +5V: now also C34.1, J10.9, J11.9, J13.9 (Pin_9), U2.28 (VCC)
- net A0: now also U8.9 (A7), J13.19 (Pin_19), U2.10 (A0); no longer U8.2 (A0)
- net A1: now also U8.8 (A6), J13.20 (Pin_20), U2.9 (A1); no longer U8.3 (A1)
- net A10: now also U10.7 (A5), J13.29 (Pin_29), U2.21 (A10); no longer U10.4 (A2)
- net A11: now also U10.6 (A4), J13.30 (Pin_30), U2.23 (A11); no longer U10.5 (A3)
- net A12: now also U10.5 (A3), J13.31 (Pin_31), U2.2 (A12); no longer U10.6 (A4)
- net A13: now also J2.40, J8.40, U10.4 (A2), J13.37 (Pin_37); no longer J2.21, J8.21, U10.9 (A7)
- net A14: now also J2.39, J8.39, U10.3 (A1), J13.38 (Pin_38); no longer J2.22, J8.22, U10.8 (A6)
- net A15: now also J2.38, J8.38, U10.2 (A0), J13.39 (Pin_39); no longer J2.23, J8.23, U10.7 (A5)
- net A2: now also U8.7 (A5), J13.21 (Pin_21), U2.8 (A2); no longer U8.4 (A2)
- net A3: now also U8.6 (A4), J13.22 (Pin_22), U2.7 (A3); no longer U8.5 (A3)
- net A4: now also U8.5 (A3), J13.23 (Pin_23), U2.6 (A4); no longer U8.6 (A4)
- net A5: now also U8.4 (A2), J13.24 (Pin_24), U2.5 (A5); no longer U8.7 (A5)
- net A6: now also U8.3 (A1), J13.25 (Pin_25), U2.4 (A6); no longer U8.8 (A6)
- net A7: now also U8.2 (A0), J13.26 (Pin_26), U2.3 (A7); no longer U8.9 (A7)
- net A8: now also U10.9 (A7), J13.27 (Pin_27), U2.25 (A8); no longer U10.2 (A0)
- net A9: now also U10.8 (A6), J13.28 (Pin_28), U2.24 (A9); no longer U10.3 (A1)
- net AP21: now also J22.40, J24.40; no longer J22.21, J24.21
- net AP22: now also J22.39, J24.39; no longer J22.22, J24.22
- net AP23: now also J22.38, J24.38; no longer J22.23, J24.23
- net AP24: now also J22.37, J24.37; no longer J22.24, J24.24
- net AP25: now also J22.36, J24.36; no longer J22.25, J24.25
- net AP26: now also J22.35, J24.35; no longer J22.26, J24.26
- net AP27: now also J22.34, J24.34; no longer J22.27, J24.27
- net AP28: now also J22.33, J24.33; no longer J22.28, J24.28
- net AP29: now also J22.32, J24.32; no longer J22.29, J24.29
- net AP30: now also J22.31, J24.31; no longer J22.30, J24.30
- net AP31: now also J22.30, J24.30; no longer J22.31, J24.31
- net AP32: now also J22.29, J24.29; no longer J22.32, J24.32
- net AP33: now also J22.28, J24.28; no longer J22.33, J24.33
- net AP34: now also J22.27, J24.27; no longer J22.34, J24.34
- net AP35: now also J22.26, J24.26; no longer J22.35, J24.35
- net AP36: now also J22.25, J24.25; no longer J22.36, J24.36
- net AP37: now also J22.24, J24.24; no longer J22.37, J24.37
- net AP38: now also J22.23, J24.23; no longer J22.38, J24.38
- net AP39: now also J22.22, J24.22; no longer J22.39, J24.39
- net BP21: now also J26.40, J29.40; no longer J26.21, J29.21
- net BP22: now also J26.39, J29.39; no longer J26.22, J29.22
- net BP23: now also J26.38, J29.38; no longer J26.23, J29.23
- net BP24: now also J26.37, J29.37; no longer J26.24, J29.24
- net BP25: now also J26.36, J29.36; no longer J26.25, J29.25
- net BP26: now also J26.35, J29.35; no longer J26.26, J29.26
- net BP27: now also J26.34, J29.34; no longer J26.27, J29.27
- net BP28: now also J26.33, J29.33; no longer J26.28, J29.28
- net BP29: now also J26.32, J29.32; no longer J26.29, J29.29
- net BP30: now also J26.31, J29.31; no longer J26.30, J29.30
- net BP31: now also J26.30, J29.30; no longer J26.31, J29.31
- net BP32: now also J26.29, J29.29; no longer J26.32, J29.32
- net BP33: now also J26.28, J29.28; no longer J26.33, J29.33
- net BP34: now also J26.27, J29.27; no longer J26.34, J29.34
- net BP35: now also J26.26, J29.26; no longer J26.35, J29.35
- net BP36: now also J26.25, J29.25; no longer J26.36, J29.36
- net BP37: now also J26.24, J29.24; no longer J26.37, J29.37
- net BP38: now also J26.23, J29.23; no longer J26.38, J29.38
- net BP39: now also J26.22, J29.22; no longer J26.39, J29.39
- net BP40: now also J26.21, J29.21; no longer J26.40, J29.40
- net CP33: now also J8.28; no longer J1.33 (Pin_33), J2.33, J3.33 (Pin_33), J8.33
- net CP36: now also J8.25; no longer J1.36 (Pin_36), J2.36, J3.36 (Pin_36), J8.36
- net CP38: now also J8.23; no longer J1.38 (Pin_38), J2.38, J3.38 (Pin_38), J8.38
- net CP39: now also J2.22, J8.22; no longer J2.39, J8.39
- net CP5: no longer J1.5 (Pin_5), J2.5, J3.5 (Pin_5)
- net CP6: no longer J1.6 (Pin_6), J2.6, J3.6 (Pin_6)
- net D0: now also J2.30, J8.30, U12.18 (B0), J13.10 (Pin_10), U2.11 (I/O0); no longer J2.31, J8.31, U12.11 (B7)
- net D0_33: now also U12.2 (A0), U5.31 (48_IOR49B); no longer U12.9 (A7), U5.21 (52_IOR39A)
- net D1: now also J2.31, J8.31, U12.17 (B1), J13.11 (Pin_11), U2.12 (I/O1); no longer J2.30, J8.30, U12.12 (B6)
- net D1_33: now also U12.3 (A1), U5.29 (49_IOR49A); no longer U12.8 (A6), U5.22 (53_IOR38B)
- net D2: now also J2.32, J8.32, U12.16 (B2), J13.12 (Pin_12), U2.13 (I/O2); no longer J2.29, J8.29, U12.13 (B5)
- net D2_33: now also U12.4 (A2), U5.28 (86_IOT4A); no longer U12.7 (A5), U5.23 (71_IOT44A)
- net D3: now also J2.33, J8.33, U12.15 (B3), J13.13 (Pin_13), U2.15 (I/O3); no longer J2.28, J8.28, U12.14 (B4)
- net D3_33: now also U12.5 (A3), U5.27 (79_IOT27B); no longer U12.6 (A4), U5.24 (72_IOT40B)
- net D4: now also J2.34, J8.34, U12.14 (B4), J13.14 (Pin_14), U2.16 (I/O4); no longer J2.27, J8.27, U12.15 (B3)
- net D4_33: now also U12.6 (A4), U5.24 (72_IOT40B); no longer U12.5 (A3), U5.27 (79_IOT27B)
- net D5: now also J2.35, J8.35, U12.13 (B5), J13.15 (Pin_15), U2.17 (I/O5); no longer J2.26, J8.26, U12.16 (B2)
- net D5_33: now also U12.7 (A5), U5.23 (71_IOT44A); no longer U12.4 (A2), U5.28 (86_IOT4A)
- net D6: now also J2.36, J8.36, U12.12 (B6), J13.16 (Pin_16), U2.18 (I/O6); no longer J2.25, J8.25, U12.17 (B1)
- net D6_33: now also U12.8 (A6), U5.22 (53_IOR38B); no longer U12.3 (A1), U5.29 (49_IOR49A)
- net D7: now also J2.37, J8.37, U12.11 (B7), J13.17 (Pin_17), U2.19 (I/O7); no longer J2.24, J8.24, U12.18 (B0)
- net D7_33: now also U12.9 (A7), U5.21 (52_IOR39A); no longer U12.2 (A0), U5.31 (48_IOR49B)
- net DP4: now also J10.4, J11.4
- net DP5: now also J10.5, J11.5
- net E: now also J2.27, J8.27, J13.6 (Pin_6); no longer J2.34, J8.34
- net GND: now also C34.2, J10.8, J11.8, J13.33 (Pin_33), J13.34 (Pin_34), U2.14 (GND)
- net PIA0: now also J10.14, J11.14
- net PIA1: now also J10.15, J11.15
- net Q: now also J2.26, J8.26, J13.7 (Pin_7), JP1.1 (A); no longer J2.35, J8.35
- net R/~{W}: now also J2.29, J8.29, J13.18 (Pin_18), U2.27 (*WE); no longer J2.32, J8.32
- net S0: now also J10.1, J11.1
- net S1: now also J10.2, J11.2
- net S2: now also J10.3, J11.3
- net ~{CART}: now also J13.8 (Pin_8), JP1.2 (B)
- net ~{CTS}: now also J10.13, J11.13, J13.32 (Pin_32)
- net ~{HALT}: now also J2.21, J8.21, J13.3 (Pin_3); no longer J2.40, J8.40
- net ~{HS}: now also J22.21, J24.21; no longer J22.40, J24.40
- net ~{NMI}: now also J13.4 (Pin_4)
- net ~{RESET}: now also J2.24, J8.24, J13.5 (Pin_5); no longer J2.37, J8.37
- net ~{SCS}: now also J10.16, J11.16, J13.36 (Pin_36), U2.20 (*CE), U2.22 (*OE)
- net ~{SLENB}: now also J10.6, J11.6, J13.40 (Pin_40)
- net AP18 renamed AP19
- new net SND: J13.35 (Pin_35)
- no-connect marks 21 -> 40
Other:
- moved on the sheet: U22

Commit message: final PCB v1.0.0
Parts:
- D1, D3: value BAT54H,111 -> SD103BW
Other:
- note added: "HBDOS-CART"
- moved on the sheet: C11, C13, C14, C15, C16, C22, C23, C24, C25, C26, C27, C28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

Commit message: gerber
Parts:
- removed H1, H2, H3, H4: MountingHole, MountingHole:MountingHole_3mm, symbol Mechanical:MountingHole

Commit message: fixes
Parts:
- added C10, C12: 1800pF, Capacitor_SMD:C_0805_2012Metric_Pad1.18x1.45mm_HandSolder, symbol Device:C
- added R19: 47K, Resistor_SMD:R_0805_2012Metric_Pad1.20x1.40mm_HandSolder, symbol Device:R
Connections:
- net +5V: now also U2.27 (*WE), R19.1
- net GND: now also U2.20 (*CE), C10.2, C12.2
- net ROW0: no longer D1.2 (A)
- net ROW1: no longer D3.2 (A)
- net ROW2: now also D3.2 (A), C12.1
- net ROW3: now also D1.2 (A), C10.1
- net R/~{W}: now also R19.2; no longer U2.27 (*WE)
- net ~{CTS}: now also U2.22 (*OE)
- net ~{HALT}: no longer Q9.3
- net ~{RESET}: now also Q9.3
- net ~{SCS}: no longer U2.20 (*CE), U2.22 (*OE)

Commit message: Prepare to release public
Parts:
- removed J10: 74LS138_ZIF, FPGA_Common:CONN_CF4216FH0R0-05-NH_CVI, symbol FPGA_Common:CF4216FH0R0-05-NH
- removed J11: 74LS138_ZIF_SOCKET, FPGA_Common:CONN_CF4216FH0R0-05-NH_CVI, symbol FPGA_Common:CF4216FH0R0-05-NH
- removed J12: PIA1_SOCKET, Package_DIP:DIP-40_W15.24mm_Socket, symbol Connector_Generic:Conn_02x20_Counter_Clockwise
- removed J2: CPU_SOCKET_ZIF, FPGA_Common:CONN_CF4240FH0R0-05-NH_CVI, symbol FPGA_Common:CF4240FH0R0-05-NH
- removed J22: PIA0_SOCKET_ZIF, FPGA_Common:CONN_CF4240FH0R0-05-NH_CVI, symbol FPGA_Common:CF4240FH0R0-05-NH
- removed J24: PIA0_ZIF, FPGA_Common:CONN_CF4240FH0R0-05-NH_CVI, symbol FPGA_Common:CF4240FH0R0-05-NH
- removed J26: PIA1_SOCKET_ZIF, FPGA_Common:CONN_CF4240FH0R0-05-NH_CVI, symbol FPGA_Common:CF4240FH0R0-05-NH
- removed J29: PIA1_ZIF, FPGA_Common:CONN_CF4240FH0R0-05-NH_CVI, symbol FPGA_Common:CF4240FH0R0-05-NH
- removed J3: CPU_SOCKET, Package_DIP:DIP-40_W15.24mm_Socket, symbol Connector_Generic:Conn_02x20_Counter_Clockwise
- removed J8: CPU_ZIF, FPGA_Common:CONN_CF4240FH0R0-05-NH_CVI, symbol FPGA_Common:CF4240FH0R0-05-NH
- removed J9: PIA0_SOCKET, Package_DIP:DIP-40_W15.24mm_Socket, symbol Connector_Generic:Conn_02x20_Counter_Clockwise
- added J10: PIA1_OUT, Connector_PinHeader_2.54mm:PinHeader_1x02_P2.54mm_Vertical, symbol Connector_Generic:Conn_01x02
- added J14: PIA0_IN, Connector_PinHeader_2.54mm:PinHeader_1x03_P2.54mm_Vertical, symbol Connector_Generic:Conn_01x03
- added J15: PIA1_IN, Connector_PinHeader_2.54mm:PinHeader_1x02_P2.54mm_Vertical, symbol Connector_Generic:Conn_01x02
- added J2: ADDRMUX_OUT, Connector_PinHeader_2.54mm:PinHeader_1x06_P2.54mm_Vertical, symbol Connector_Generic:Conn_01x06
- added J3: ADDRMUX_IN, Connector_PinHeader_2.54mm:PinHeader_1x06_P2.54mm_Vertical, symbol Connector_Generic:Conn_01x06
- added J8: PIA0_OUT, Connector_PinHeader_2.54mm:PinHeader_1x03_P2.54mm_Vertical, symbol Connector_Generic:Conn_01x03
- J1, J4, J5: footprint Package_DIP:DIP-40_W15.24mm_Socket -> FPGA_Common:DIP-40_W15.24mm-OVERSIZED
- J28: value ADDRMUX_SOCKET -> ADDRMUX; footprint Package_DIP:DIP-16_W7.62mm_Socket -> FPGA_Common:DIP-16_W7.62mm-OVERSIZED
- U1: value SN74HC138PWR -> 74HC138
- U10, U11, U12, U8: value SN74LVC245AN -> 74LVC245
- U9: value SN74HC245PWR -> 74HC245
Connections:
- net A0: now also U8.2 (A0); no longer U8.9 (A7)
- net A1: now also U8.3 (A1); no longer U8.8 (A6)
- net A11: now also U10.8 (A6); no longer U10.6 (A4)
- net A12: now also U10.9 (A7); no longer U10.5 (A3)
- net A2: now also U8.4 (A2); no longer U8.7 (A5)
- net A3: now also U8.5 (A3); no longer U8.6 (A4)
- net A4: now also U8.6 (A4); no longer U8.5 (A3)
- net A5: now also U8.7 (A5); no longer U8.4 (A2)
- net A6: now also U8.8 (A6); no longer U8.3 (A1)
- net A7: now also U8.9 (A7); no longer U8.2 (A0)
- net A8: now also U10.5 (A3); no longer U10.9 (A7)
- net A9: now also U10.6 (A4); no longer U10.8 (A6)
- net DATADIR: now also J2.6 (Pin_6), J3.6 (Pin_6)
- net KEYINT: now also J14.1 (Pin_1), J8.3 (Pin_3)
- net ROW2: no longer C12.1
- net ROW3: no longer C10.1
- net S0: now also J2.1 (Pin_1), J3.1 (Pin_1)
- net S1: now also J2.2 (Pin_2), J3.2 (Pin_2)
- net S2: now also J2.3 (Pin_3), J3.3 (Pin_3)
- net SERNT: now also J10.1 (Pin_1), J15.1 (Pin_1)
- net ~{CART}: now also J10.2 (Pin_2), J15.2 (Pin_2)
- net ~{DATAEN}: now also J2.5 (Pin_5), J3.5 (Pin_5)
- net ~{FS}: now also J14.3 (Pin_3), J8.2 (Pin_2)
- net ~{HS}: now also J14.2 (Pin_2), J8.1 (Pin_1)
- net ~{SLENB}: now also J2.4 (Pin_4), J3.4 (Pin_4)
- net at D3.1 (K), J23.2 (Pin_2): now also C12.1
- net at D1.1 (K), J23.1 (Pin_1): now also C10.1
- net CP39 renamed TSC
- net DP4 renamed G2A
- net DP5 renamed G2B
- no-connect marks 40 -> 22
Other:
- note added: "ADDRMUX DAUGHTERBOARD"
- note added: "MAIN BOARD"
- note added: "PIA0 (SC67331) DAUGHTERBOARD"
- note added: "PIA1 (MC6821) DAUGHTERBOARD"
- note removed: "ADDRMUX DISPLACER"
- note removed: "CPU DISPLACER"
- note removed: "PIA0 DISPLACER"
- note removed: "PIA1 DISPLACER"
- moved on the sheet: C1, C10, C12, C2, C3, C32, C33, C34, C4, C5, C6, C7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
