File: kicad/CoCoTANG.kicad_pcb (KiCad board)
At the start: 2 copper layers, 213.4 x 88.1 mm, 105 parts, among them J1 CPU, J10 PIA0, J11 PIA1, J12 PIA1_SOCKET, J13 ADDRMUX_SOCKET, J14 PIA0, J15 PIA1, J16 VDG_IN, J17 AV_IN, J18 CMP_IN, J19 VDG_OUT, J2 ADDRMUX, J20 AV_OUT, J21 CMP_OUT, J3 CPU_SOCKET, J4 PIA0, J5 PIA1, J6 ADDRMUX, J7 AV_HEADER, J8 ADDRMUX, J9 PIA0_SOCKET, Q1 2N3904, Q2 2N3904, Q3 2N3904, Q4 MMBT3904, Q5 MMBT3904, Q6 MMBT3904, Q7 MMBT3904, Q8 MMBT3904, Q9 MMBT3904, U10 SN74LVC245AN, U11 SN74LVC245AN, U12 SN74LVC245AN, U3 74HC139, U5 Tang_Nano_20k, U7 74HC30, U8 SN74LVC245AN, U9 SN74LVC245AN

Commit message: changes
Parts:
- removed J19: VDG_OUT, Connector_PinHeader_2.54mm:PinHeader_1x05_P2.54mm_Vertical
- added C32: 104, Capacitor_SMD:C_0805_2012Metric_Pad1.18x1.45mm_HandSolder, F.Cu at (0.00, 0.00)
- added D1, D3: BAT54H,111, Diode_SMD:D_SOD-123F, F.Cu at (0.00, 0.00)
- added J22: 74HC11, Package_SO:TSSOP-14_4.4x5mm_P0.65mm, F.Cu at (0.00, 0.00)
- added J23: TRG, Connector_PinHeader_2.54mm:PinHeader_1x02_P2.54mm_Vertical, F.Cu at (0.00, 0.00)
- added J24: VDG_SOCKET, Package_DIP:DIP-40_W15.24mm_Socket, F.Cu at (0.00, 0.00)
- added J25: AUDIO_OUT, Connector_PinHeader_2.54mm:PinHeader_1x02_P2.54mm_Vertical, F.Cu at (0.00, 0.00)
- added RV1: VREF, FPGA_Common:PVG3G_BRN, F.Cu at (0.00, 0.00)
Connections:
- net CHA_VDG renamed CLRA
- net CHB_VDG renamed CLRB
- J8 pad 4: ~{MRD} -> ~{DATAEN}
Routing:
- net GND: track 492.0 -> 561.1 mm
- net +5V: track 91.7 -> 143.2 mm
- net ROW0: track 8.46 -> 47.8 mm, vias 0 -> 1
- net ROW1: track 6.99 -> 44.1 mm, vias 0 -> 1
- net CHB_33: track 5.81 -> 41.6 mm
- net CHA_33: track 5.45 -> 31.7 mm
- net Y_33: track 80.2 -> 103.1 mm
- net ~{ROM}: track 0.00 -> 20.4 mm
- net AUDIO_33: track 98.6 -> 115.8 mm
- net ~{EXTROM}: track 0.00 -> 16.3 mm
- net Net-(D3-K): track 0.00 -> 12.9 mm
- net Net-(D1-K): track 0.00 -> 12.7 mm
- net ~{SLENB}: track 66.0 -> 75.9 mm
- net S2: track 36.7 -> 46.2 mm
- net Y_VDG: track 19.6 -> 10.3 mm, vias 1 -> 0
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Other:
- board size 213.4 x 88.1 mm -> 242.3 x 87.6 mm
- board text added: "ADDRMUX V1.0.1"
- board text added: "PIA0 DISPLACER V1.0.1"
- board text added: "TRG"
- board text added: "VDG V1.0.1"
- board text removed: "ADDRMUX V1.0.0"
- board text removed: "CH.A"
- board text removed: "CH.B"
- board text removed: "PIA0 DISPLACER V1.0.0"
- board text removed: "VDG V1.0.0"

Commit message: new board
Parts:
- removed C10, C12: 22uF, Capacitor_SMD:C_0805_2012Metric_Pad1.18x1.45mm_HandSolder
- removed C17, C18, C19: 68pF, Capacitor_SMD:C_0805_2012Metric_Pad1.18x1.45mm_HandSolder
- removed C20: 4.7uF, Capacitor_SMD:C_0805_2012Metric_Pad1.18x1.45mm_HandSolder
- removed C21: 6.8nF, Capacitor_SMD:C_0805_2012Metric_Pad1.18x1.45mm_HandSolder
- removed J10, J14: PIA0, Connector_PinHeader_2.54mm:PinHeader_1x03_P2.54mm_Vertical
- removed J11, J15: PIA1, Connector_PinHeader_2.54mm:PinHeader_1x02_P2.54mm_Vertical
- removed J13: ADDRMUX_SOCKET, Package_DIP:DIP-16_W7.62mm_Socket
- removed J16: VDG_IN, Connector_PinHeader_2.54mm:PinHeader_1x06_P2.54mm_Vertical
- removed J25: AUDIO_OUT, Connector_PinHeader_2.54mm:PinHeader_1x02_P2.54mm_Vertical
- removed R19, R20, R21: 100, Resistor_SMD:R_0805_2012Metric_Pad1.20x1.40mm_HandSolder
- removed RV1: VREF, FPGA_Common:PVG3G_BRN
- added C33: 104, Capacitor_SMD:C_0805_2012Metric_Pad1.18x1.45mm_HandSolder, F.Cu at (0.00, 0.00)
- added J26: PIA1_SOCKET_ZIF, FPGA_Common:CONN_CF4240FH0R0-05-NH_CVI, F.Cu at (0.00, 0.00)
- added J27: ADDRMUX_SOCKET_ZIF, FPGA_Common:CONN_CF4216FH0R0-05-NH_CVI, F.Cu at (0.00, 0.00)
- added J28: ADDRMUX_SOCKET, Package_DIP:DIP-16_W7.62mm_Socket, F.Cu at (0.00, 0.00)
- added J29: PIA1_ZIF, FPGA_Common:CONN_CF4240FH0R0-05-NH_CVI, F.Cu at (0.00, 0.00)
- added J30: ADDRMUX_ZIF, FPGA_Common:CONN_CF4216FH0R0-05-NH_CVI, F.Cu at (0.00, 0.00)
- added R1, R37, R38, R39: 1K, Resistor_SMD:R_0805_2012Metric_Pad1.20x1.40mm_HandSolder, F.Cu at (0.00, 0.00)
- added U1: SN74HC138PWR, Package_SO:TSSOP-16_4.4x5mm_P0.65mm, F.Cu at (0.00, 0.00)
- added U22: 74HC11, Package_SO:TSSOP-14_4.4x5mm_P0.65mm, F.Cu at (0.00, 0.00)
- C14: value 680pF -> 470pF
- J2: value ADDRMUX -> CPU_SOCKET_ZIF; footprint Connector_PinHeader_2.54mm:PinHeader_1x05_P2.54mm_Vertical -> FPGA_Common:CONN_CF4240FH0R0-05-NH_CVI
- J22: value 74HC11 -> PIA0_SOCKET_ZIF; footprint Package_SO:TSSOP-14_4.4x5mm_P0.65mm -> FPGA_Common:CONN_CF4240FH0R0-05-NH_CVI
- J24: value VDG_SOCKET -> PIA0_ZIF; footprint Package_DIP:DIP-40_W15.24mm_Socket -> FPGA_Common:CONN_CF4240FH0R0-05-NH_CVI
- J6: value ADDRMUX -> CLK; footprint Package_DIP:DIP-16_W7.62mm_Socket -> Connector_PinSocket_2.54mm:PinSocket_1x01_P2.54mm_Vertical
- J8: value ADDRMUX -> CPU_ZIF; footprint Connector_PinHeader_2.54mm:PinHeader_1x05_P2.54mm_Vertical -> FPGA_Common:CONN_CF4240FH0R0-05-NH_CVI
- Q1, Q2, Q3: value 2N3904 -> MMBT3904-TP; footprint Package_TO_SOT_SMD:SOT-23 -> FPGA_Common:SOT-23_MCC
- Q4, Q5, Q6, Q7, Q8, Q9: value MMBT3904 -> MMBT3904-TP; footprint Package_TO_SOT_SMD:SOT-23 -> FPGA_Common:SOT-23_MCC
- R17: value 100K -> 1K
- U9: value SN74LVC245AN -> SN74HC245PWR
Connections:
- net HALT_33 renamed RESET_33
- C2 pad 1: +3.3V -> +5V
- J1 pad 24: D0 -> D7
- J1 pad 25: D1 -> D6
- J1 pad 26: D2 -> D5
- J1 pad 27: D3 -> D4
- J1 pad 28: D4 -> D3
- J1 pad 29: D5 -> D2
- J1 pad 30: D6 -> D1
- J1 pad 31: D7 -> D0
- J2 pad 1: S0 -> GND
- J2 pad 2: S1 -> ~{NMI}
- J2 pad 3: S2 -> ~{IRQ}
- J2 pad 4: ~{MRD} -> ~{FIRQ}
- J2 pad 5: ~{SLENB} -> CP5
- J22 pad 1: ~{MRD} -> GND
- J22 pad 10: unconnected-(J22-Pin_10-Pad10) -> AP10
- J22 pad 11: unconnected-(J22-Pin_11-Pad11) -> AP11
- J22 pad 12: ~{DATAEN} -> AP12
- J22 pad 13: ~{EXTROM} -> AP13
- J22 pad 14: +5V -> AP14
- J22 pad 2: ~{ROM} -> ROW0
- J22 pad 3: unconnected-(J22-Pin_3-Pad3) -> ROW1
- J22 pad 4: unconnected-(J22-Pin_4-Pad4) -> ROW2
- J22 pad 5: unconnected-(J22-Pin_5-Pad5) -> ROW3
- J22 pad 6: unconnected-(J22-Pin_6-Pad6) -> ROW4
- J22 pad 7: GND -> ROW5
- J22 pad 8: unconnected-(J22-Pin_8-Pad8) -> ROW6
- J22 pad 9: unconnected-(J22-Pin_9-Pad9) -> AP9
- J24 pad 10: CLRB -> AP10
- J24 pad 11: CLRA -> AP11
- J24 pad 12: unconnected-(J24-Pin_12-Pad12) -> AP12
- J24 pad 13: unconnected-(J24-Pin_13-Pad13) -> AP13
- J24 pad 14: unconnected-(J24-Pin_14-Pad14) -> AP14
- J24 pad 15: unconnected-(J24-Pin_15-Pad15) -> AP15
- J24 pad 16: unconnected-(J24-Pin_16-Pad16) -> AP16
- J24 pad 17: +5V -> AP17
- J24 pad 18: unconnected-(J24-Pin_18-Pad18) -> ~{FS}
- J24 pad 19: unconnected-(J24-Pin_19-Pad19) -> AP18
- J24 pad 2: unconnected-(J24-Pin_2-Pad2) -> ROW0
- J24 pad 20: unconnected-(J24-Pin_20-Pad20) -> +5V
- J24 pad 21: unconnected-(J24-Pin_21-Pad21) -> AP21
- J24 pad 22: unconnected-(J24-Pin_22-Pad22) -> AP22
- J24 pad 23: unconnected-(J24-Pin_23-Pad23) -> AP23
- J24 pad 24: unconnected-(J24-Pin_24-Pad24) -> AP24
- J24 pad 25: unconnected-(J24-Pin_25-Pad25) -> AP25
- J24 pad 26: unconnected-(J24-Pin_26-Pad26) -> AP26
- J24 pad 27: unconnected-(J24-Pin_27-Pad27) -> AP27
- J24 pad 28: Y_VDG -> AP28
- J24 pad 29: unconnected-(J24-Pin_29-Pad29) -> AP29
- J24 pad 3: unconnected-(J24-Pin_3-Pad3) -> ROW1
- J24 pad 30: unconnected-(J24-Pin_30-Pad30) -> AP30
- J24 pad 31: unconnected-(J24-Pin_31-Pad31) -> AP31
- J24 pad 32: unconnected-(J24-Pin_32-Pad32) -> AP32
- J24 pad 33: unconnected-(J24-Pin_33-Pad33) -> AP33
- J24 pad 34: unconnected-(J24-Pin_34-Pad34) -> AP34
- J24 pad 35: unconnected-(J24-Pin_35-Pad35) -> AP35
- J24 pad 36: unconnected-(J24-Pin_36-Pad36) -> AP36
- J24 pad 37: unconnected-(J24-Pin_37-Pad37) -> AP37
- J24 pad 38: unconnected-(J24-Pin_38-Pad38) -> AP38
- J24 pad 39: unconnected-(J24-Pin_39-Pad39) -> AP39
- J24 pad 4: unconnected-(J24-Pin_4-Pad4) -> ROW2
- J24 pad 40: unconnected-(J24-Pin_40-Pad40) -> ~{HS}
- J24 pad 5: unconnected-(J24-Pin_5-Pad5) -> ROW3
- J24 pad 6: unconnected-(J24-Pin_6-Pad6) -> ROW4
- J24 pad 7: unconnected-(J24-Pin_7-Pad7) -> ROW5
- J24 pad 8: unconnected-(J24-Pin_8-Pad8) -> ROW6
- J24 pad 9: CHB -> AP9
- J3 pad 24: D0 -> D7
- J3 pad 25: D1 -> D6
- J3 pad 26: D2 -> D5
- J3 pad 27: D3 -> D4
- J3 pad 28: D4 -> D3
- J3 pad 29: D5 -> D2
- J3 pad 30: D6 -> D1
- J3 pad 31: D7 -> D0
- J6 pad 1: S0 -> CLK
- J7 pad 2: PB_33 -> CHR_33
- J7 pad 3: PR_33 -> CVBS_33
- J8 pad 1: S0 -> GND
- J8 pad 2: S1 -> ~{NMI}
- J8 pad 3: S2 -> ~{IRQ}
- J8 pad 4: ~{DATAEN} -> ~{FIRQ}
- J8 pad 5: ~{SLENB} -> CP5
- Q1 pad 1: GND -> Net-(Q1-Pad1)
- Q1 pad 2: Net-(Q1-B) -> Net-(Q1-Pad2)
- Q1 pad 3: ~{IRQ} -> +3.3V
- Q2 pad 1: GND -> Net-(Q2-Pad1)
- Q2 pad 2: Net-(Q2-B) -> Net-(Q2-Pad2)
- Q2 pad 3: ~{HALT} -> +3.3V
- Q3 pad 1: GND -> Net-(Q3-Pad1)
- Q3 pad 2: Net-(Q3-B) -> Net-(Q3-Pad2)
- Q3 pad 3: ~{FIRQ} -> +3.3V
- Q4 pad 1: Net-(Q4-B) -> Net-(Q4-Pad1)
- Q4 pad 2: Net-(Q4-E) -> Net-(Q4-Pad2)
- Q5 pad 1: Net-(Q5-B) -> Net-(Q5-Pad1)
- Q5 pad 2: Net-(Q5-E) -> Net-(Q5-Pad2)
- Q6 pad 1: Net-(Q6-B) -> Net-(Q6-Pad1)
- Q6 pad 2: Net-(Q6-E) -> Net-(Q6-Pad2)
- Q7 pad 1: Net-(Q7-B) -> Net-(Q7-Pad1)
- Q7 pad 2: Net-(Q7-E) -> GND
- Q7 pad 3: +3.3V -> ~{IRQ}
- Q8 pad 1: Net-(Q8-B) -> Net-(Q8-Pad1)
- Q8 pad 2: Net-(Q8-E) -> GND
- Q8 pad 3: +3.3V -> ~{FIRQ}
- Q9 pad 1: Net-(Q9-B) -> Net-(Q9-Pad1)
- Q9 pad 2: Net-(Q9-E) -> GND
- Q9 pad 3: +3.3V -> ~{HALT}
- R10 pad 1: Net-(Q4-E) -> Net-(Q2-Pad2)
- R11 pad 1: Net-(Q5-E) -> Net-(Q4-Pad2)
- R11 pad 2: Net-(C10-Pad1) -> PB_RCA
- R12 pad 1: Net-(Q6-E) -> Net-(Q5-Pad2)
- R12 pad 2: Net-(C12-Pad1) -> PR_RCA
- R13 pad 2: Net-(Q7-E) -> Net-(Q1-Pad2)
- R14 pad 2: Net-(Q8-E) -> Net-(Q3-Pad2)
- R15 pad 1: Net-(Q9-E) -> Net-(Q6-Pad2)
- R16 pad 1: AUDIO_33 -> Net-(Q5-Pad2)
- R16 pad 2: Net-(C20-Pad1) -> GND
- R17 pad 1: GND -> Net-(Q2-Pad2)
- R17 pad 2: AUDIO_RCA -> GND
- R25 pad 2: Net-(Q7-B) -> Net-(Q1-Pad1)
- R26 pad 1: Net-(Q7-B) -> Net-(Q1-Pad1)
- R27 pad 2: Net-(Q8-B) -> Net-(Q3-Pad1)
- R28 pad 1: Net-(Q8-B) -> Net-(Q3-Pad1)
- R29 pad 2: Net-(Q9-B) -> Net-(Q6-Pad1)
- R3 pad 1: Net-(Q1-B) -> Net-(Q7-Pad1)
- R30 pad 1: Net-(Q9-B) -> Net-(Q6-Pad1)
- R31 pad 2: Net-(Q4-B) -> Net-(Q2-Pad1)
- R32 pad 1: Net-(Q4-B) -> Net-(Q2-Pad1)
- R33 pad 2: Net-(Q5-B) -> Net-(Q4-Pad1)
- R34 pad 1: Net-(Q5-B) -> Net-(Q4-Pad1)
- R35 pad 2: Net-(Q6-B) -> Net-(Q5-Pad1)
- R36 pad 1: Net-(Q6-B) -> Net-(Q5-Pad1)
- R5 pad 1: Net-(Q2-B) -> Net-(Q9-Pad1)
- R7 pad 1: Net-(Q3-B) -> Net-(Q8-Pad1)
- U12 pad 1: R/~{W} -> DATADIR
- U12 pad 19: ~{MRD} -> ~{DATAEN}
- U5 pad 18: FIRQ_33 -> CVBS_33
- U5 pad 3: E_33 -> FIRQ_33
- U5 pad 32: PR_33 -> E_33
- U5 pad 33: PB_33 -> CHR_33
- U9 pad 11: unconnected-(U9-B7-Pad11) -> CLK
- U9 pad 20: +3.3V -> +5V
- U9 pad 9: unconnected-(U9-A7-Pad9) -> AUDIO_33
Routing:
- net GND: track 561.1 -> 0.00 mm, vias 10 -> 0
- net +3.3V: track 291.2 -> 0.00 mm, vias 13 -> 0
- net +5V: track 143.2 -> 0.00 mm
- net AUDIO_33: track 115.8 -> 0.00 mm, vias 2 -> 0
- net ~{HALT}: track 111.2 -> 0.00 mm, vias 3 -> 0
- net Y_33: track 103.1 -> 0.00 mm, vias 1 -> 0
- net R/~{W}: track 97.1 -> 0.00 mm, vias 1 -> 0
- net ~{HS}: track 89.2 -> 0.00 mm, vias 1 -> 0
- net KEYINT: track 88.9 -> 0.00 mm
- net ~{FS_33}: track 85.4 -> 0.00 mm, vias 1 -> 0
- net ~{HS_33}: track 85.1 -> 0.00 mm, vias 1 -> 0
- net ~{RESET}: track 84.0 -> 0.00 mm
- net MSEL1_33: track 81.7 -> 0.00 mm, vias 1 -> 0
- net SERNT: track 80.8 -> 0.00 mm, vias 1 -> 0
- net E_33: track 79.6 -> 0.00 mm, vias 1 -> 0
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- removed copper zone on B.Cu, net GND
- removed copper zone on F.Cu, net GND
Other:
- board size 242.3 x 87.6 mm -> 172.7 x 92.2 mm
- board text added: "74LS138"
- board text added: "COCOTANG V1.00 2026 LUIS ANTONIOSI"
- board text added: "COMPONENT / RGB 1.1"
- board text added: "COMPONENT VIDEO 1.1"
- board text added: "CPU"
- board text added: "PB/B"
- board text added: "PR/R"
- board text added: "TANG NANO 20K"
- board text added: "Y/G"
- board text removed: "1"
- board text removed: "A/V IN"
- board text removed: "A/V OUT"
- board text removed: "ADDRMUX"
- board text removed: "ADDRMUX V1.0.1"
- board text removed: "CHROMA"
- board text removed: "COMP V1.0.0"
- board text removed: "CPU SOCKET V1.0.0"
- board text removed: "CVBS"
- board text removed: "CocoTANG v1.0.0 2026 LUIS ANTONIOSI"
- board text removed: "MC6809E"
- board text removed: "PB"
- board text removed: "PIA0 DISPLACER V1.0.1"
- board text removed: "PIA1 DISPLACER V1.0.0"
- board text removed: "PR"
- board text removed: "SVIDEO V1.0.0"
- board text removed: "TANG Nano 20K"
- board text removed: "TRG"
- board text removed: "VDG V1.0.1"
- board text removed: "Y"

Commit message: fixes
Parts:
- removed J27: ADDRMUX_SOCKET_ZIF, FPGA_Common:CONN_CF4216FH0R0-05-NH_CVI
- removed J30: ADDRMUX_ZIF, FPGA_Common:CONN_CF4216FH0R0-05-NH_CVI
- added C34: 104, Capacitor_SMD:C_0805_2012Metric_Pad1.18x1.45mm_HandSolder, F.Cu at (0.00, 0.00)
- added H1, H2, H3, H4: MountingHole, MountingHole:MountingHole_3mm, F.Cu at (0.00, 0.00)
- added J10: 74LS138_ZIF, FPGA_Common:CONN_CF4216FH0R0-05-NH_CVI, F.Cu at (0.00, 0.00)
- added J11: 74LS138_ZIF_SOCKET, FPGA_Common:CONN_CF4216FH0R0-05-NH_CVI, F.Cu at (0.00, 0.00)
- added J13: CoCo_Cart, FPGA_Common:COCO_CART, F.Cu at (0.00, 0.00)
- added JP1: Jumper_2_Open, Jumper:SolderJumper-2_P1.3mm_Open_Pad1.0x1.5mm, F.Cu at (0.00, 0.00)
- added U2: AT28C64B-15PU, FPGA_Common:28P6_ATM, F.Cu at (0.00, 0.00)
Connections:
- net AP18 renamed AP19
- J1 pad 33: CP33 -> unconnected-(J1-Pin_33-Pad33)
- J1 pad 36: CP36 -> unconnected-(J1-Pin_36-Pad36)
- J1 pad 38: CP38 -> unconnected-(J1-Pin_38-Pad38)
- J1 pad 5: CP5 -> unconnected-(J1-Pin_5-Pad5)
- J1 pad 6: CP6 -> unconnected-(J1-Pin_6-Pad6)
- J2 pad 21: A13 -> ~{HALT}
- J2 pad 22: A14 -> CP39
- J2 pad 23: A15 -> unconnected-(J2-Pad23)
- J2 pad 24: D7 -> ~{RESET}
- J2 pad 25: D6 -> unconnected-(J2-Pad25)
- J2 pad 26: D5 -> Q
- J2 pad 27: D4 -> E
- J2 pad 28: D3 -> unconnected-(J2-Pad28)
- J2 pad 29: D2 -> R/~{W}
- J2 pad 30: D1 -> D0
- J2 pad 31: D0 -> D1
- J2 pad 32: R/~{W} -> D2
- J2 pad 33: CP33 -> D3
- J2 pad 34: E -> D4
- J2 pad 35: Q -> D5
- J2 pad 36: CP36 -> D6
- J2 pad 37: ~{RESET} -> D7
- J2 pad 38: CP38 -> A15
- J2 pad 39: CP39 -> A14
- J2 pad 40: ~{HALT} -> A13
- J2 pad 5: CP5 -> unconnected-(J2-Pad5)
- J2 pad 6: CP6 -> unconnected-(J2-Pad6)
- J22 pad 21: AP21 -> ~{HS}
- J22 pad 22: AP22 -> AP39
- J22 pad 23: AP23 -> AP38
- J22 pad 24: AP24 -> AP37
- J22 pad 25: AP25 -> AP36
- J22 pad 26: AP26 -> AP35
- J22 pad 27: AP27 -> AP34
- J22 pad 28: AP28 -> AP33
- J22 pad 29: AP29 -> AP32
- J22 pad 30: AP30 -> AP31
- J22 pad 31: AP31 -> AP30
- J22 pad 32: AP32 -> AP29
- J22 pad 33: AP33 -> AP28
- J22 pad 34: AP34 -> AP27
- J22 pad 35: AP35 -> AP26
- J22 pad 36: AP36 -> AP25
- J22 pad 37: AP37 -> AP24
- J22 pad 38: AP38 -> AP23
- J22 pad 39: AP39 -> AP22
- J22 pad 40: ~{HS} -> AP21
- J24 pad 21: AP21 -> ~{HS}
- J24 pad 22: AP22 -> AP39
- J24 pad 23: AP23 -> AP38
- J24 pad 24: AP24 -> AP37
- J24 pad 25: AP25 -> AP36
- J24 pad 26: AP26 -> AP35
- J24 pad 27: AP27 -> AP34
- J24 pad 28: AP28 -> AP33
- J24 pad 29: AP29 -> AP32
- J24 pad 30: AP30 -> AP31
- J24 pad 31: AP31 -> AP30
- J24 pad 32: AP32 -> AP29
- J24 pad 33: AP33 -> AP28
- J24 pad 34: AP34 -> AP27
- J24 pad 35: AP35 -> AP26
- J24 pad 36: AP36 -> AP25
- J24 pad 37: AP37 -> AP24
- J24 pad 38: AP38 -> AP23
- J24 pad 39: AP39 -> AP22
- J24 pad 40: ~{HS} -> AP21
- J26 pad 21: BP21 -> BP40
- J26 pad 22: BP22 -> BP39
- J26 pad 23: BP23 -> BP38
- J26 pad 24: BP24 -> BP37
- J26 pad 25: BP25 -> BP36
- J26 pad 26: BP26 -> BP35
- J26 pad 27: BP27 -> BP34
- J26 pad 28: BP28 -> BP33
- J26 pad 29: BP29 -> BP32
- J26 pad 30: BP30 -> BP31
- J26 pad 31: BP31 -> BP30
- J26 pad 32: BP32 -> BP29
- J26 pad 33: BP33 -> BP28
- J26 pad 34: BP34 -> BP27
- J26 pad 35: BP35 -> BP26
- J26 pad 36: BP36 -> BP25
- J26 pad 37: BP37 -> BP24
- J26 pad 38: BP38 -> BP23
- J26 pad 39: BP39 -> BP22
- J26 pad 40: BP40 -> BP21
- J29 pad 21: BP21 -> BP40
- J29 pad 22: BP22 -> BP39
- J29 pad 23: BP23 -> BP38
- J29 pad 24: BP24 -> BP37
- J29 pad 25: BP25 -> BP36
- J29 pad 26: BP26 -> BP35
- J29 pad 27: BP27 -> BP34
- J29 pad 28: BP28 -> BP33
- J29 pad 29: BP29 -> BP32
- J29 pad 30: BP30 -> BP31
- J29 pad 31: BP31 -> BP30
- J29 pad 32: BP32 -> BP29
- J29 pad 33: BP33 -> BP28
- J29 pad 34: BP34 -> BP27
- J29 pad 35: BP35 -> BP26
- J29 pad 36: BP36 -> BP25
- J29 pad 37: BP37 -> BP24
- J29 pad 38: BP38 -> BP23
- J29 pad 39: BP39 -> BP22
- J29 pad 40: BP40 -> BP21
- J3 pad 33: CP33 -> unconnected-(J3-Pin_33-Pad33)
- J3 pad 36: CP36 -> unconnected-(J3-Pin_36-Pad36)
- J3 pad 38: CP38 -> unconnected-(J3-Pin_38-Pad38)
- J3 pad 5: CP5 -> unconnected-(J3-Pin_5-Pad5)
- J3 pad 6: CP6 -> unconnected-(J3-Pin_6-Pad6)
- J8 pad 21: A13 -> ~{HALT}
- J8 pad 22: A14 -> CP39
- J8 pad 23: A15 -> CP38
- J8 pad 24: D7 -> ~{RESET}
- J8 pad 25: D6 -> CP36
- J8 pad 26: D5 -> Q
- J8 pad 27: D4 -> E
- J8 pad 28: D3 -> CP33
- J8 pad 29: D2 -> R/~{W}
- J8 pad 30: D1 -> D0
- J8 pad 31: D0 -> D1
- J8 pad 32: R/~{W} -> D2
- J8 pad 33: CP33 -> D3
- J8 pad 34: E -> D4
- J8 pad 35: Q -> D5
- J8 pad 36: CP36 -> D6
- J8 pad 37: ~{RESET} -> D7
- J8 pad 38: CP38 -> A15
- J8 pad 39: CP39 -> A14
- J8 pad 40: ~{HALT} -> A13
- U10 pad 2: A8 -> A15
- U10 pad 3: A9 -> A14
- U10 pad 4: A10 -> A13
- U10 pad 5: A11 -> A12
- U10 pad 6: A12 -> A11
- U10 pad 7: A15 -> A10
- U10 pad 8: A14 -> A9
- U10 pad 9: A13 -> A8
- U12 pad 11: D0 -> D7
- U12 pad 12: D1 -> D6
- U12 pad 13: D2 -> D5
- U12 pad 14: D3 -> D4
- U12 pad 15: D4 -> D3
- U12 pad 16: D5 -> D2
- U12 pad 17: D6 -> D1
- U12 pad 18: D7 -> D0
- U12 pad 2: D7_33 -> D0_33
- U12 pad 3: D6_33 -> D1_33
- U12 pad 4: D5_33 -> D2_33
- U12 pad 5: D4_33 -> D3_33
- U12 pad 6: D3_33 -> D4_33
- U12 pad 7: D2_33 -> D5_33
- U12 pad 8: D1_33 -> D6_33
- U12 pad 9: D0_33 -> D7_33
- U5 pad 21: D0_33 -> D7_33
- U5 pad 22: D1_33 -> D6_33
- U5 pad 23: D2_33 -> D5_33
- U5 pad 24: D3_33 -> D4_33
- U5 pad 27: D4_33 -> D3_33
- U5 pad 28: D5_33 -> D2_33
- U5 pad 29: D6_33 -> D1_33
- U5 pad 31: D7_33 -> D0_33
- U8 pad 2: A0 -> A7
- U8 pad 3: A1 -> A6
- U8 pad 4: A2 -> A5
- U8 pad 5: A3 -> A4
- U8 pad 6: A4 -> A3
- U8 pad 7: A5 -> A2
- U8 pad 8: A6 -> A1
- U8 pad 9: A7 -> A0
Routing:
- net GND: track 0.00 -> 390.7 mm, vias 0 -> 6
- net +5V: track 0.00 -> 162.1 mm
- net +3.3V: track 0.00 -> 100.0 mm, vias 0 -> 3
- net R/~{W}: track 0.00 -> 75.7 mm
- net A10: track 0.00 -> 72.5 mm
- net ~{SCS}: track 0.00 -> 66.4 mm
- net A12: track 0.00 -> 54.4 mm
- net Y_RCA: track 0.00 -> 53.8 mm, vias 0 -> 1
- net A7: track 0.00 -> 48.4 mm
- net AUDIO_33: track 0.00 -> 47.6 mm, vias 0 -> 1
- net D1: track 0.00 -> 44.5 mm
- net D0: track 0.00 -> 44.0 mm
- net A4: track 0.00 -> 42.8 mm
- net A11: track 0.00 -> 42.6 mm
- net A6: track 0.00 -> 42.4 mm
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- added copper zone on B.Cu, net GND
- added copper zone on F.Cu, net GND
Other:
- board size 172.7 x 92.2 mm -> 227.6 x 77.9 mm
- board text added: "A/V"
- board text added: "CHR"
- board text added: "CVBS"
- board text added: "TRG2"
- board text added: "Y"

Commit message: final PCB v1.0.0
Routing:
- net GND: track 390.7 -> 1157.5 mm, vias 6 -> 10
- net +5V: track 162.1 -> 487.4 mm, vias 0 -> 4
- net +3.3V: track 100.0 -> 412.5 mm, vias 3 -> 9
- net ~{HS}: track 28.3 -> 248.7 mm, vias 0 -> 1
- net AUDIO_33: track 47.6 -> 201.1 mm
- net ~{HALT}: track 28.4 -> 174.5 mm, vias 0 -> 1
- net ROW0: track 17.3 -> 150.2 mm
- net ~{FS}: track 23.5 -> 154.5 mm, vias 0 -> 2
- net ~{FIRQ}: track 13.4 -> 144.0 mm, vias 0 -> 2
- net Q: track 31.8 -> 160.9 mm, vias 0 -> 2
- net ~{SLENB}: track 7.54 -> 135.5 mm, vias 0 -> 3
- net ~{IRQ}: track 15.2 -> 143.1 mm, vias 0 -> 1
- net ROW1: track 15.2 -> 142.9 mm
- net SERNT: track 10.2 -> 137.6 mm, vias 0 -> 1
- net E: track 16.2 -> 142.6 mm, vias 0 -> 1
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Other:
- outline, holes or cut-outs redrawn

Commit message: gerber
Parts:
- removed H1, H2, H3, H4: MountingHole, MountingHole:MountingHole_3mm
Other:
- outline, holes or cut-outs redrawn

Commit message: Prepare to release public
Parts:
- removed J11: 74LS138_ZIF_SOCKET, FPGA_Common:CONN_CF4216FH0R0-05-NH_CVI
- removed J12: PIA1_SOCKET, Package_DIP:DIP-40_W15.24mm_Socket
- removed J22: PIA0_SOCKET_ZIF, FPGA_Common:CONN_CF4240FH0R0-05-NH_CVI
- removed J24: PIA0_ZIF, FPGA_Common:CONN_CF4240FH0R0-05-NH_CVI
- removed J26: PIA1_SOCKET_ZIF, FPGA_Common:CONN_CF4240FH0R0-05-NH_CVI
- removed J29: PIA1_ZIF, FPGA_Common:CONN_CF4240FH0R0-05-NH_CVI
- removed J9: PIA0_SOCKET, Package_DIP:DIP-40_W15.24mm_Socket
- added C10, C12: 1800pF, Capacitor_SMD:C_0805_2012Metric_Pad1.18x1.45mm_HandSolder, F.Cu at (0.00, 0.00)
- added J14: PIA0_IN, Connector_PinHeader_2.54mm:PinHeader_1x03_P2.54mm_Vertical, F.Cu at (0.00, 0.00)
- added J15: PIA1_IN, Connector_PinHeader_2.54mm:PinHeader_1x02_P2.54mm_Vertical, F.Cu at (0.00, 0.00)
- added R19: 47K, Resistor_SMD:R_0805_2012Metric_Pad1.20x1.40mm_HandSolder, F.Cu at (0.00, 0.00)
- D1, D3: value BAT54H,111 -> SD103BW
- J1, J4, J5: footprint Package_DIP:DIP-40_W15.24mm_Socket -> FPGA_Common:DIP-40_W15.24mm-OVERSIZED
- J10: value 74LS138_ZIF -> PIA1_OUT; footprint FPGA_Common:CONN_CF4216FH0R0-05-NH_CVI -> Connector_PinHeader_2.54mm:PinHeader_1x02_P2.54mm_Vertical
- J2: value CPU_SOCKET_ZIF -> ADDRMUX_OUT; footprint FPGA_Common:CONN_CF4240FH0R0-05-NH_CVI -> Connector_PinHeader_2.54mm:PinHeader_1x06_P2.54mm_Vertical
- J28: value ADDRMUX_SOCKET -> ADDRMUX; footprint Package_DIP:DIP-16_W7.62mm_Socket -> FPGA_Common:DIP-16_W7.62mm-OVERSIZED
- J3: value CPU_SOCKET -> ADDRMUX_IN; footprint Package_DIP:DIP-40_W15.24mm_Socket -> Connector_PinHeader_2.54mm:PinHeader_1x06_P2.54mm_Vertical
- J8: value CPU_ZIF -> PIA0_OUT; footprint FPGA_Common:CONN_CF4240FH0R0-05-NH_CVI -> Connector_PinHeader_2.54mm:PinHeader_1x03_P2.54mm_Vertical
- U1: value SN74HC138PWR -> 74HC138
- U10, U11, U12, U8: value SN74LVC245AN -> 74LVC245
- U9: value SN74HC245PWR -> 74HC245
Connections:
- D1 pad 2: ROW0 -> ROW3
- D3 pad 2: ROW1 -> ROW2
- J1 pad 39: CP39 -> TSC
- J10 pad 1: S0 -> SERNT
- J10 pad 2: S1 -> ~{CART}
- J2 pad 1: GND -> S0
- J2 pad 2: ~{NMI} -> S1
- J2 pad 3: ~{IRQ} -> S2
- J2 pad 4: ~{FIRQ} -> ~{SLENB}
- J2 pad 5: unconnected-(J2-Pad5) -> ~{DATAEN}
- J2 pad 6: unconnected-(J2-Pad6) -> DATADIR
- J28 pad 4: DP4 -> G2A
- J28 pad 5: DP5 -> G2B
- J3 pad 1: GND -> S0
- J3 pad 2: ~{NMI} -> S1
- J3 pad 3: ~{IRQ} -> S2
- J3 pad 4: ~{FIRQ} -> ~{SLENB}
- J3 pad 5: unconnected-(J3-Pin_5-Pad5) -> ~{DATAEN}
- J3 pad 6: unconnected-(J3-Pin_6-Pad6) -> DATADIR
- J8 pad 1: GND -> ~{HS}
- J8 pad 2: ~{NMI} -> ~{FS}
- J8 pad 3: ~{IRQ} -> KEYINT
- Q9 pad 3: ~{HALT} -> ~{RESET}
- U1 pad 4: DP4 -> G2A
- U1 pad 5: DP5 -> G2B
- U10 pad 5: A12 -> A8
- U10 pad 6: A11 -> A9
- U10 pad 8: A9 -> A11
- U10 pad 9: A8 -> A12
- U2 pad 20: ~{SCS} -> GND
- U2 pad 22: ~{SCS} -> ~{CTS}
- U2 pad 27: R/~{W} -> +5V
- U8 pad 2: A7 -> A0
- U8 pad 3: A6 -> A1
- U8 pad 4: A5 -> A2
- U8 pad 5: A4 -> A3
- U8 pad 6: A3 -> A4
- U8 pad 7: A2 -> A5
- U8 pad 8: A1 -> A6
- U8 pad 9: A0 -> A7
Routing:
- net GND: track 1157.5 -> 897.6 mm, vias 10 -> 24
- net +5V: track 487.4 -> 294.6 mm, vias 4 -> 3
- net ROW0: track 150.2 -> 7.25 mm
- net ROW1: track 142.9 -> 6.46 mm
- net ROW6: track 135.7 -> 14.4 mm, vias 1 -> 0
- net CP39: track 120.4 -> 0.00 mm, vias 1 -> 0
- net BP30: track 118.5 -> 0.00 mm
- net BP31: track 116.2 -> 0.00 mm
- net ROW4: track 122.2 -> 6.73 mm
- net ~{IRQ}: track 143.1 -> 28.3 mm, vias 1 -> 0
- net BP32: track 114.5 -> 0.00 mm
- net Q: track 160.9 -> 47.7 mm, vias 2 -> 1
- net ~{FIRQ}: track 144.0 -> 30.9 mm, vias 2 -> 0
- net BP33: track 112.8 -> 0.00 mm
- net BP34: track 111.0 -> 0.00 mm
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Other:
- board size 227.6 x 77.9 mm -> 215.9 x 85.1 mm
- board text added: "CVBS VIDEO 1.1"
- board text removed: "74LS138"
- board text removed: "A/V"
- board text removed: "COMPONENT VIDEO 1.1"
- board text removed: "CPU"
- board text removed: "PIA0"
- board text removed: "PIA1"
- board text removed: "TANG NANO 20K"
- board text removed: "TRG2"
